File: hardware/dc-electronic-load.kicad_pcb (KiCad board)
At the start: 2 copper layers, 92 parts, among them M1 Mounting Hole, M2 Mounting Hole, M3 Mounting Hole, M4 Mounting Hole, M5 Heat Sink (RA-T2X-38E), M6 Power Entry Connector, M7 Enclosure (8.36x9.11x3.15), M8 Fan (50mm x 10mm), M9 Fan Guard, P1 BELFUSE-08B0-1X1T-06-F, P2 FTDI-PLUG, P3 SWD, P8 FAN, U1 LD1086V33, U10 TSV631ILT, U11 BUK954R8-60E,127, U2 ENC28J60, U3 STM32-64PIN, U4 TIREF30XX, U5 SST25VF032B-S2A, U6 25AA02EXXX-XOT, U7 MCP3204, U8 MCP49X1, U9 FQT7N10LTF, X1 25MHz, X2 32.768kHZ, X3 8MHz

Commit message: pcb 2014-09-30
Parts:
- removed C23: 100uF, klib:CAPAE660X790N
- added C28: 0.1uF, klib:CAPC2012X100N, F.Cu at (130.9, 70.0)
- added C29: 0.1uF, klib:CAPC2012X100N, F.Cu at (140.8, 83.9)
- added C30: 0.1uF, klib:CAPC2012X100N, F.Cu at (147.3, 73.4)
- added C31: 0.1uF, klib:CAPC2012X100N, F.Cu at (130.2, 79.5)
- added C32: 0.1uF, klib:CAPC2012X100N, F.Cu at (147.3, 80.1)
- added D3: 24V, klib:DIOM5226X220N, F.Cu at (158.1, 88.4)
- added P10: TEMP1, klib:JST-B2B-XH-A, F.Cu at (116.0, 103.2)
- added P11: TEMP2, klib:JST-B2B-XH-A, F.Cu at (171.7, 106.3)
- added P12: LOAD-GND, klib:PAD205P, F.Cu at (144.4, 135.8)
- added P13: VSENSE, klib:JST-B2B-XH-A, F.Cu at (151.5, 86.9)
- added P4: ENCODER, klib:JST-B5B-XH-A, F.Cu at (103.8, 128.7)
- added P5: BUTTONS, klib:JST-B5B-XH-A, F.Cu at (114.0, 86.8)
- added P6: POWER, klib:TECONN-2-1445050-2, F.Cu at (194.9, 70.2)
- added P7: LCD, klib:SHDRV26W100P254_2X13_4052X880X910P, F.Cu at (106.3, 109.7)
- added P9: LOAD-VCC, klib:PAD205P, F.Cu at (144.4, 93.2)
- added R36: 1K, klib:RESC2012X100N, F.Cu at (156.8, 85.3)
- P8: footprint klib:EMPTY -> klib:JST-B2B-XH-A
- R20: value 820 -> 1K
- R23: value 9K1 -> 10K
- moved U11 111.4 mm to (144.4, 105.9)
- moved R10 101.1 mm to (108.2, 120.2)
- moved U5 95.8 mm to (158.7, 80.8)
- moved U10 92.4 mm to (141.0, 112.2), turned to 90 degrees
- moved R9 92.2 mm to (108.2, 127.7)
- moved M7 89.2 mm to (110.0, 67.7)
- moved R12 89.0 mm to (108.2, 122.7), turned to 180 degrees
- moved U6 88.7 mm to (155.3, 75.1)
- moved M6 88.5 mm to (111.0, 67.7)
- moved M8 87.7 mm to (112.0, 67.7)
- moved M9 87.0 mm to (113.0, 67.7)
- moved R13 86.0 mm to (116.7, 115.7), turned to 180 degrees
- moved R34 80.6 mm to (111.7, 103.0), turned to 90 degrees
- moved R11 79.3 mm to (108.2, 125.2), turned to 180 degrees
- moved C27 79.2 mm to (112.5, 115.7)
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Connections:
- R23 pad 1: Net-(P9-Pad1) -> Net-(D3-Pad2)
Routing:
- net +3.3V: track 0.00 -> 422.0 mm, vias 0 -> 10
- net GNDPWR: track 0.00 -> 218.7 mm, vias 0 -> 39
- net /ISENSE: track 0.00 -> 195.8 mm
- net /SPI2MOSI: track 0.00 -> 92.0 mm, vias 0 -> 4
- net /SPI2SCK: track 0.00 -> 89.7 mm, vias 0 -> 2
- net Net-(R19-Pad2): track 0.00 -> 84.2 mm, vias 0 -> 4
- net /DACCS: track 0.00 -> 78.4 mm, vias 0 -> 2
- net /SPI2MISO: track 0.00 -> 72.2 mm, vias 0 -> 4
- net /FAN: track 0.00 -> 67.5 mm, vias 0 -> 2
- net /ADCCS: track 0.00 -> 66.3 mm, vias 0 -> 4
- net /ENCODERBUTTON: track 0.00 -> 66.0 mm, vias 0 -> 5
- net /ENCODERA: track 0.00 -> 65.1 mm, vias 0 -> 4
- net /TEMP1: track 0.00 -> 64.1 mm, vias 0 -> 4
- net /LCDDATA1: track 0.00 -> 62.6 mm, vias 0 -> 4
- net /LCDDATA0: track 0.00 -> 60.8 mm, vias 0 -> 5
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- added copper zone on B.Cu, net GNDPWR
- added copper zone on F.Cu, net GNDPWR
Other:
- board outline added: 106.8 x 73.5 mm
- net class Default: clearance 0.254 -> 0.2032; trace_width 0.254 -> 0.2032; via_dia 0.889 -> 0.6858; via_drill 0.635 -> 0.3302
- net class load added: clearance 0.508, trace_width 2.54, via_dia 0.6858, via_drill 0.3302
- net class power added: clearance 0.508, trace_width 1.27, via_dia 0.889, via_drill 0.635
- net class powersmall added: clearance 0.2032, trace_width 0.254, via_dia 0.6858, via_drill 0.3302
- rule trace_clearance: 0.254 -> 0.2032
- rule trace_min: 0.254 -> 0.1524
- rule via_min_drill: 0.508 -> 0.3302
- rule via_min_size: 0.889 -> 0.6858
- board text added: "+"
- board text added: "+3.3V SWCLK GND SWDIO nRST"
- board text added: "-"
- board text added: "2014-09-30"
- board text added: "4-6V"
- board text added: "A B C D GND"
- board text added: "BUTTONS"
- board text added: "DC Electronic Load"
- board text added: "DEBUG"
- board text added: "ENCODER"
- board text added: "FAN"
- board text added: "GND"
- board text added: "Joe Ferner"
- board text added: "LOAD+"
- board text added: "LOAD-"
- board text added: "OLED"
- board text added: "POWER"
- board text added: "RX TX"
- board text added: "SWD"
- board text added: "TEMP1"
- board text added: "TEMP2"
- board text added: "VSENSE"
- board text added: "https://github.com/joeferner/dc-electronic-load"
