File: hardware/buttons.kicad_pcb (KiCad board)
At the start: 2 copper layers, 104 x 8.1 mm, 7 parts, among them M1 Mounting Hole, M2 Mounting Hole, P1 P05

Commit message: buttons 2014-11-09
Other:
- board text added: "OLED Button Bar 2014-11-09"
Changed lines of the file:
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@@
     (area 95.949999 96.349999 200.050001 104.550001)
     (thickness 1.6)
-    (drawings 4)
+    (drawings 5)
     (tracks 32)
     (zones 0)
@@
     (visible_elements FFFFFF7F)
     (pcbplotparams
-      (layerselection 0x00030_80000001)
-      (usegerberextensions false)
-      (excludeedgelayer true)
+      (layerselection 0x010f0_80000001)
+      (usegerberextensions true)
+      (excludeedgelayer false)
       (linewidth 0.100000)
       (plotframeref false)
@@
       (outputformat 1)
       (mirror false)
-      (drillshape 1)
+      (drillshape 0)
       (scaleselection 1)
-      (outputdirectory ""))
+      (outputdirectory buttons-2014-11-09/))
   )
   (net 0 "")
@@
       (effects (font (size 0.6 0.6) (thickness 0.1)))
     )
-    (fp_text value "Mounting Hole" (at 0 0) (layer F.SilkS)
+    (fp_text value "Mounting Hole" (at 0 0) (layer F.SilkS) hide
       (effects (font (size 0.6 0.6) (thickness 0.1)))
     )
@@
       (effects (font (size 0.6 0.6) (thickness 0.1)))
     )
-    (fp_text value "Mounting Hole" (at 0 0) (layer F.SilkS)
+    (fp_text value "Mounting Hole" (at 0 0) (layer F.SilkS) hide
       (effects (font (size 0.6 0.6) (thickness 0.1)))
     )
@@
       (effects (font (size 0.6 0.6) (thickness 0.1)) (justify mirror))
     )
-    (fp_text value P05 (at -3.139 2.381 90) (layer B.SilkS)
+    (fp_text value P05 (at -3.139 2.381 90) (layer B.SilkS) hide
       (effects (font (size 0.6 0.6) (thickness 0.1)) (justify mirror))
     )
@@
       (net 5 GNDPWR))
   )
+  (gr_text "OLED Button Bar 2014-11-09" (at 145 100) (layer B.SilkS)
+    (effects (font (size 1.5 1.5) (thickness 0.3)) (justify mirror))
+  )
   (gr_line (start 96 104.5) (end 96 96.4) (angle 90) (layer Edge.Cuts) (width 0.1))
